File: 514_pcb/514_pcb.kicad_pcb (KiCad board)
At the start: 2 copper layers, 60.5 x 52 mm, 5 parts, among them SW1 SW_SPDT

Commit message: updates
Parts:
- added C1: C_Polarized, Resistor_SMD:R_0603_1608Metric_Pad0.98x0.95mm_HandSolder, F.Cu at (130.6, 100.0)
- added D1: APA102, LED_SMD:LED_RGB_5050-6, F.Cu at (131.6, 93.3)
- BT1: footprint Connector_JST:JST_NV_B02P-NV_1x02_P5.00mm_Vertical -> Connector_JST:JST_JWPF_B02B-JWPF-SK-R_1x02_P2.00mm_Vertical
- R1: value R -> R = 10k
- SW1: footprint Button_Switch_SMD:SW_SPDT_PCM12 -> Connector_PinHeader_2.54mm:PinHeader_1x03_P2.54mm_Vertical
- U1: footprint SeeedXiao:XIAO_ESP32_SENSE -> Seeed Studio XIAO Series Library:XIAO-ESP32S3-DIP
Connections:
- U1 pad 10: Net-(MK1-VDD) -> unconnected-(U1-GPIO8/D9/A9/MISO-Pad10)
- U1 pad 11: unconnected-(U1-GPIO9_A10_D10_COPI-Pad11) -> Net-(D1-DI)
- U1 pad 12: unconnected-(U1-GPIO8_A9_D9_CIPO-Pad12) -> Net-(MK1-VDD)
- U1 pad 13: unconnected-(U1-GPIO7_A8_D8_SCK-Pad13) -> GND
- U1 pad 14: unconnected-(U1-GPIO44_D7_RX-Pad14) -> Net-(SW1-A)
- U1 pad 8: Net-(SW1-A) -> unconnected-(U1-U0RXD/D7/RX-Pad8)
- U1 pad 9: GND -> Net-(D1-CI)
Routing:
- net GND: track 0.00 -> 21.1 mm, vias 0 -> 2
- net Net-(BT1-+): track 0.00 -> 14.2 mm
