File: 514_pcb/514_pcb.kicad_sch (KiCad schematic)
At the start: 4 parts, among them SW1 SW_SPDT, U1 LAFVIN-ESP32-WROOM-32

Commit message: updates
Parts:
- removed U1: LAFVIN-ESP32-WROOM-32, RF_Module:ESP32-WROOM-32, symbol RF_Module:LAFVIN-ESP32-WROOM-32
- added BT1: Battery_Cell, Connector_JST:JST_JWPF_B02B-JWPF-SK-R_1x02_P2.00mm_Vertical, symbol Device:Battery_Cell
- added U1: ~, SeeedXiao:XIAO_ESP32_SENSE, symbol SeeedXiao:XIAO_ESP32_SENSE
- R1: value R -> R = 10k
- SW1: footprint Button_Switch_THT:SW_PUSH-12mm -> Connector_PinHeader_2.54mm:PinHeader_1x03_P2.54mm_Vertical
Connections:
- net GND: now also MK1.2 (SEL), BT1.2 (-), U1.9 (GND)
- net at MK1.1 (WS): now also U1.5 (GPIO4_A3_D3_SDA)
- net at MK1.4 (BCLK): now also U1.6 (GPIO6_A5_D5_SCL)
- net at MK1.5 (VDD): now also U1.10 (3V3)
- net at MK1.6 (DATA), R1.1: now also U1.7 (GPIO43_TX_D6)
- net at SW1.1 (A): now also U1.8 (5V)
- net at SW1.2 (B): now also BT1.1 (+)
- no-connect marks 25 -> 9
Other:
- note added: "Diyun Lu"
- moved on the sheet: MK1, R1, SW1

Commit message: updates
Parts:
- added C1: C_Polarized, Resistor_SMD:R_0603_1608Metric_Pad0.98x0.95mm_HandSolder, symbol Device:C_Polarized
- added D1: APA102, LED_SMD:LED_RGB_5050-6, symbol LED:APA102
- U1: footprint SeeedXiao:XIAO_ESP32_SENSE -> Seeed Studio XIAO Series Library:XIAO-ESP32S3-DIP; symbol SeeedXiao:XIAO_ESP32_SENSE -> Seeed_Studio_XIAO_Series:XIAO-ESP32-S3-DIP
Connections:
- net GND: now also U1.13 (GND), C1.2, D1.3 (GND); no longer U1.9 (GND)
- net at U1.10 (GPIO8/D9/A9/MISO): no longer MK1.5 (VDD)
- net at U1.11 (GPIO9/D10/A10/MOSI): now also D1.1 (DI)
- net at U1.12 (VCC_3V3): now also MK1.5 (VDD)
- net at U1.14 (VBUS): now also SW1.1 (A)
- net at U1.8 (U0RXD/D7/RX): no longer SW1.1 (A)
- net at BT1.1 (+), SW1.2 (B): now also C1.1, D1.4 (VCC)
- new net: D1.2 (CI), U1.9 (GPIO7/D8/A8/SCK)
- no-connect marks 9 -> 7
Other:
- moved on the sheet: BT1, MK1, R1, SW1
